Commit message: 3D建图有重影版

File: src/27_rc_simulation/livox_laser_simulation_RO2/urdf/mid360.xacro (robot description, xacro)
@@ -5,4 +5,6 @@
   <xacro:property name="laser_max_range" value="200.0"/>
   <xacro:property name="samples" value="30000"/>
+<!--        -->
+  <xacro:property name="downsample" value="5"/>
   <xacro:property name="resolution" value="0.002"/>
   <xacro:property name="noise_mean" value="0.0"/>
@@ -21,8 +23,11 @@
   <xacro:macro name="mid360" params="name:='' parent:= 'base_link' topic:='mid360' *origin ">
     <link name="${name}">
+    <!---->
+      <xacro:box_inertia m="${mass}" w="${width}" h="${height}" d="${length}"/>
+      <!---->
       <visual>
         <origin xyz="0.025 -0.0265 -0.025" rpy="${pi/2} 0 ${pi}"/>
         <geometry>
-          <mesh filename="model://mid360.stl" scale="0.0008 0.0008 0.0008"/>
+          <mesh filename="package://ros2_livox_simulation/meshes/mid360.stl" scale="0.0008 0.0008 0.0008"/>
         </geometry>
       </visual>
@@ -33,10 +38,33 @@
       <xacro:insert_block name="origin"/>
     </joint>
+    <!-- 保留传感器 link，避免固定关节合并后影响底盘碰撞与插件挂载。 -->
+    <gazebo reference="${name}_joint">
+      <preserveFixedJoint>true</preserveFixedJoint>
+    </gazebo>
     <gazebo reference="${name}">
       <sensor type="ray" name="${name}">
         <pose>0 0 0 0 0 0</pose>
-        <visualize>true</visualize>
+        <always_on>true</always_on>
+        <visualize>false</visualize>
         <update_rate>10</update_rate>
+        <!---->
+        <!-- 标准 ray sensor 驱动更新回调；真实的非重复射线由下面插件生成。 -->
+        <ray>
+          <scan>
+            <horizontal>
+              <samples>2</samples><resolution>1</resolution>
+              <min_angle>0</min_angle><max_angle>${2*M_PI}</max_angle>
+            </horizontal>
+          </scan>
+          <range>
+            <min>${laser_min_range}</min><max>${laser_max_range}</max>
+            <resolution>${resolution}</resolution>
+          </range>
+        </ray>
+        <!---->
         <plugin name="${name}_plugin" filename="libros2_livox.so">
+        <!---->
+          <frame_name>${name}</frame_name>
+        <!---->
           <ray>
             <scan>
@@ -67,5 +95,5 @@
           <visualize>false</visualize>
           <samples>${samples}</samples>
-          <downsample>1</downsample>
+          <downsample>${downsample}</downsample>
           <csv_file_name>$(find ros2_livox_simulation)/scan_mode/mid360.csv</csv_file_name>
           <topic>${topic}</topic>

File: src/27_rc_simulation/robocon2027_gazebo/urdf/simulation_waking_robot.xacro (robot description, xacro)
@@ -14,4 +14,8 @@
   <xacro:arg name="xyz" default="0.12 0.0 0.175" />
   <xacro:arg name="rpy" default="0 0 0" />
+  <!-- 第一阶段可关闭 Livox，避免雷达驱动依赖阻止基础小车启动。 -->
+  <xacro:arg name="use_livox" default="true" />
+  <!-- 二维沿用 Gazebo TF；三维入口关闭它，由 FAST-LIO 定位。 -->
+  <xacro:arg name="publish_odom_tf" default="true" />
   <link name="dummy"/>
   <link name="base_link">
@@ -52,6 +56,4 @@
       </geometry>
     </collision>
-    <mu1>0.5</mu1>
-    <mu2>0.5</mu2>
     <xacro:default_inertial mass="0.5"/>
   </link>
@@ -69,6 +71,4 @@
       </geometry>
     </collision>
-    <mu1>0.5</mu1>
-    <mu2>0.5</mu2>
     <xacro:default_inertial mass="0.5"/>
   </link>
@@ -86,6 +86,4 @@
       </geometry>
     </collision>
-    <mu1>0.5</mu1>
-    <mu2>0.5</mu2>
     <xacro:default_inertial mass="0.5"/>
   </link>
@@ -103,6 +101,4 @@
       </geometry>
     </collision>
-    <mu1>0.5</mu1>
-    <mu2>0.5</mu2>
     <xacro:default_inertial mass="0.5"/>
   </link>
@@ -115,5 +111,4 @@
   <joint name="base_to_wheel2" type="continuous">
     <axis xyz="0 0 1" />
-    <anchor xyz="0 0 0" />
     <limit effort="100" velocity="100" />
     <parent link="base_link"/>
@@ -169,13 +164,17 @@
   <gazebo reference="wheel_1">
     <material>Gazebo/Red</material>
+    <mu1>0.5</mu1><mu2>0.5</mu2>
   </gazebo>
   <gazebo reference="wheel_2">
     <material>Gazebo/Black</material>
+    <mu1>0.5</mu1><mu2>0.5</mu2>
   </gazebo>
   <gazebo reference="wheel_3">
     <material>Gazebo/Red</material>
+    <mu1>0.5</mu1><mu2>0.5</mu2>
   </gazebo>
   <gazebo reference="wheel_4">
     <material>Gazebo/Black</material>
+    <mu1>0.5</mu1><mu2>0.5</mu2>
   </gazebo>
   <gazebo reference="imu_link">
@@ -188,5 +187,6 @@
   <!-- https://github.com/ros-simulation/gazebo_ros_pkgs/wiki/ROS-2-Migration:-Planar-Move -->
   <gazebo>
-    <plugin name="mecanum_controller" filename="libgazebo_ros_planar_move.so">
+    <!-- 沿用平面速度控制，但保留竖直速度，让重力和地面碰撞决定接地高度。 -->
+    <plugin name="mecanum_controller" filename="librc_planar_move.so">
       <ros>
         <!-- Add a namespace -->
@@ -200,10 +200,13 @@
       <!-- Set odom publish rate -->
       <publish_rate>10</publish_rate>
+      <cmd_timeout>0.5</cmd_timeout>
       <!-- Set if odom required -->
-      <publish_odom>false</publish_odom>
-      <publish_odom_tf>false</publish_odom_tf>
+      <publish_odom>true</publish_odom>
+      <publish_odom_tf>$(arg publish_odom_tf)</publish_odom_tf>
       <!-- Frame IDs -->
       <odometry_frame>odom</odometry_frame>
-      <robot_base_frame>base_link</robot_base_frame>
+      <!-- dummy 是现有 URDF 的根，dummy_joint 已发布 dummy -> base_link。
+           在根上接 odom，避免给 base_link 同时发布两个父坐标系。 -->
+      <robot_base_frame>dummy</robot_base_frame>
       <!-- Set odom covariance -->
       <covariance_x>0.0001</covariance_x>
@@ -228,7 +231,9 @@
   </gazebo>
   <!-- Livox-Mid360  -->
-  <xacro:include filename="$(find ros2_livox_simulation)/urdf/mid360.xacro" />
-  <xacro:mid360 name="livox_frame" parent="base_link" topic="/livox/lidar">
-    <origin xyz="$(arg xyz)" rpy="$(arg rpy)" />
-  </xacro:mid360>
+  <xacro:if value="$(arg use_livox)">
+    <xacro:include filename="$(find ros2_livox_simulation)/urdf/mid360.xacro" />
+    <xacro:mid360 name="livox_frame" parent="base_link" topic="/livox/lidar">
+      <origin xyz="$(arg xyz)" rpy="$(arg rpy)" />
+    </xacro:mid360>
+  </xacro:if>
 </robot>

Commit message: Fix Gazebo chassis drift and instantaneous 3D mapping

File: src/27_rc_simulation/livox_laser_simulation_RO2/urdf/mid360.xacro (robot description, xacro)
@@ -3,5 +3,6 @@
   <xacro:property name="M_PI" value="3.1415926"/>
   <xacro:property name="laser_min_range" value="0.1"/>
-  <xacro:property name="laser_max_range" value="200.0"/>
+  <!-- Arena mapping uses the same 20 m range as FAST-LIO's det_range. -->
+  <xacro:property name="laser_max_range" value="20.0"/>
   <xacro:property name="samples" value="30000"/>
 <!--        -->

File: src/27_rc_simulation/robocon2027_gazebo/urdf/simulation_waking_robot.xacro (robot description, xacro)
@@ -196,6 +196,6 @@
         <remapping>odom:=odom</remapping>
       </ros>
-      <!-- Set control loop update rate -->
-      <update_rate>100</update_rate>
+      <!-- Apply chassis velocity every physics step; odometry stays at 10 Hz. -->
+      <update_rate>0</update_rate>
       <!-- Set odom publish rate -->
       <publish_rate>10</publish_rate>
